File: hardware/Control Board.sch (KiCad schematic (older format))
At the start: 42 parts, among them J1 Conn_FTDI, J2 SOLAR, M1 Motor_DC, Q1 IRF7105PbF, Q2 BC817W, Q3 BC817W, Q4 IRF7105PbF, SW1 SW_Push, SW2 SW_Push, SW3 SW_Push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

Commit message: Wiring up new layout
Parts:
- removed R14, R15: 10k, Resistor_SMD:R_0402_1005Metric, symbol Device:R
- added C8: 4.7uF, Capacitor_SMD:C_0402_1005Metric, symbol Device:C
- added D1, D2: SK34A, Diode_SMD:D_SMA, symbol Device:D_Schottky
- added R19: 10k, Resistor_SMD:R_0402_1005Metric, symbol Device:R
- M1: value Motor_DC -> MOTOR
- SW1: value SW_Push -> PROG
- SW2: value SW_Push -> RESET
- U1: footprint Package_DFN_QFN:Texas_S-PVQFN-N16_EP2.7x2.7mm -> Package_DFN_QFN:Texas_S-PVQFN-N16_EP2.7x2.7mm_ThermalVias
- U2: value MCP1700-3302E_SOT89 -> MCP1700
Connections:
- net +3V3: no longer J1.4 (Pin_4)
- net EN: now also SW2.2
- net GND: now also C3.1, C8.2, R19.2; no longer C3.2, U1.1 (TS)
- net IO0: now also SW1.2
- net at C2.1, U1.10 (OUT), U1.11 (OUT)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: now also C8.1
- net at U3.11 (IO8): no longer SW1.2
- net at U3.10 (IO7): no longer SW2.2
- new net: D1.2 (A), J2.1 (Pin_1)
- new net: R19.1, U1.1 (TS)
- new net: C3.2, D1.1 (K), D2.1 (K), U1.13 (IN)
- new net +5V: D2.2 (A), J1.4 (Pin_4)
- no-connect marks 23 -> 25
Other:
- moved on the sheet: C3, R1, R16
