File: hardware/Control Board.sch (KiCad schematic (older format))
At the start: 48 parts, among them J1 SOLAR, J2 Conn_FTDI, M1 MOTOR, Q1 BC817W, Q2 IRF7105PbF, Q3 BC817W, Q4 BC817W, Q5 IRF7105PbF, Q6 BC817W, SW1 PROG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

Commit message: Move to 12V, use power supply module, remove auto programmer, remove solar charger, Use ESP32-WROVER
Parts:
- removed BT1: LIPO, Connector_JST:JST_EH_B02B-EH-A_1x02_P2.50mm_Vertical, symbol Device:Battery_Cell
- removed C1, C4, C6: 10uF, Capacitor_SMD:C_0805_2012Metric, symbol Device:C
- removed C2, C3: 4.7uF, Capacitor_SMD:C_0805_2012Metric, symbol Device:C
- removed C7, C8: 0.1uF, Capacitor_SMD:C_0805_2012Metric, symbol Device:C
- removed D1, D2: SK34A, Diode_SMD:D_SMA, symbol Device:D_Schottky
- removed J2: Conn_FTDI, Connector_PinHeader_2.54mm:PinHeader_1x06_P2.54mm_Vertical, symbol Connector:Conn_01x06_Male
- removed Q3, Q4: BC817W, Package_TO_SOT_SMD:SOT-323_SC-70, symbol Transistor_BJT:BC817W
- removed R13, R14, R3: 10k, Resistor_SMD:R_0805_2012Metric, symbol Device:R
- removed R15, R16: 12k, Resistor_SMD:R_0805_2012Metric, symbol Device:R
- removed R2: 1.13k, Resistor_SMD:R_0805_2012Metric, symbol Device:R
- removed R7: 27k, Resistor_SMD:R_0805_2012Metric, symbol Device:R
- removed R8: 100k, Resistor_SMD:R_0805_2012Metric, symbol Device:R
- removed U1: BQ24075, Package_DFN_QFN:Texas_S-PVQFN-N16_EP2.7x2.7mm_ThermalVias, symbol Battery_Management:BQ24075
- removed U2: MCP1700, Package_TO_SOT_SMD:SOT-89-3, symbol Regulator_Linear:MCP1700-3302E_SOT89
- removed U3: ESP32S2-WROVER, RF_Module:ESP32-S2-WROVER, symbol esp32-wrover:ESP32S2-WROVER
- added TP1, TP10, TP2, TP3, TP4: TestPoint, TestPoint:TestPoint_Pad_1.0x1.0mm, symbol Connector:TestPoint
- added TP5: 3.3V, TestPoint:TestPoint_Pad_1.0x1.0mm, symbol Connector:TestPoint
- added TP6: RX, TestPoint:TestPoint_Pad_1.0x1.0mm, symbol Connector:TestPoint
- added TP7: TX, TestPoint:TestPoint_Pad_1.0x1.0mm, symbol Connector:TestPoint
- added TP8: IO0, TestPoint:TestPoint_Pad_1.0x1.0mm, symbol Connector:TestPoint
- added TP9: GND, TestPoint:TestPoint_Pad_1.0x1.0mm, symbol Connector:TestPoint
- added U1: Step Down, Ebay:DC Buck Step-Down Fixed Voltage Converter, symbol Ebay:DC_Buck_Step-Down_Fixed_Voltage_Converter
- added U2: ESP32-WROVER, RF_Module:ESP32-WROOM-32, symbol esp32-wrover:ESP32-WROVER
- J1: value SOLAR -> 12V
- M1: value MOTOR -> ACCUATOR
- R1: value 1.18k -> 10k
- SW1: value PROG -> RESET
- SW2: value RESET -> SW_PUSH
Connections:
- net +BATT is gone; now on net +12V: Q2.3 (S2), Q5.3 (S2), R12.1, R17.1
- net +3V3: now also R1.1, TP5.1, U1.3 (+VOUT), U2.2 (3V3)
- net GND: now also TP10.1, TP9.1, U1.2 (-VIN), U1.4 (-VOUT), U2.1 (GND), U2.15 (GND), U2.38 (GND), U2.39 (GND); no longer R1.2
- net IO0: now also TP8.1, U2.25 (IO0); no longer SW1.2
- net RX: now also TP6.1, U2.34 (RXD0)
- net TX: now also TP7.1, U2.35 (TXD0)
- net WATER_OFF: now also TP1.1, U2.30 (IO18)
- net WATER_ON: now also TP4.1, U2.31 (IO19)
- net at M1.2 (-), Q2.7 (D1), Q2.8 (D1)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: now also TP3.1
- net at M1.1 (+), Q2.5 (D2), Q2.6 (D2)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: now also TP2.1
- net +12V: now reaches J1.1 (Pin_1)
- net +12V: now also U1.1 (+VIN)
- net at SW4.2: now also R9.2, U2.9 (IO33_XTAL_32K_N); no longer R6.2
- net at SW5.2: now also R1.2, U2.10 (IO25); no longer R5.2
- net at R4.2, SW6.2: now also U2.11 (IO26)
- net at SW3.2: now also R6.2, U2.8 (IO32_XTAL_32K_P); no longer R9.2
- net EN: no longer names the net of SW2.2
- net EN: now also R5.2, U2.7 (IO35)
- new net: SW1.2, U2.3 (EN)
- no-connect marks 25 -> 20
Other:
- note added: "2.0.0"
- note added: "2021-10-06"
- note removed: "1.0.1"
- note removed: "2021-04-06"
- moved on the sheet: R4, R5, R6, R9, SW1, SW2, SW3, SW4, SW5, SW6
