File: hardware/Control Board.kicad_sch (KiCad schematic)
At the start: 52 parts, among them J1 12V, J2 SOLENOID, J3 SOLENOID, J4 SOLENOID, J5 SOLENOID, Q1 BC817W, Q2 IRF7105PbF, Q3 BC817W, Q4 BC817W, Q5 IRF7105PbF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

Commit message: Updating values of PSU
Parts:
- removed C3: 470pF, symbol Device:C
- removed D5: D_Zener, symbol Device:D_Zener
- added C3: 63uF, symbol Device:C_Polarized
- added D5: 1N5818, symbol Device:D_Schottky
- C2: value 470pF -> 433pF
- L1: value L -> 56uH
- R14: value R -> 11k
- R15: value R -> 18k
- R4: value R -> 0.2R
Connections:
- net +3V3: now also C3.1
- net GND: now also C3.2, D5.2 (A)
- net at L1.1, U1.2 (SwE): now also D5.1 (K)
Changed lines of the file:
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@@
 			)
 		)
-		(property "Value" "R"
+		(property "Value" "0.2R"
 			(at 72.39 124.46 90)
 			(effects
@@
 			)
 		)
-		(property "Value" "R"
+		(property "Value" "18k"
 			(at 114.3 143.5099 0)
 			(effects
@@
 			)
 		)
-		(property "Value" "470pF"
+		(property "Value" "433pF"
 			(at 64.77 161.2899 0)
 			(effects
@@
 	)
 	(symbol
+		(lib_id "Device:C_Polarized")
+		(at 99.06 160.02 0)
+		(unit 1)
+		(exclude_from_sim no)
+		(in_bom yes)
+		(on_board yes)
+		(dnp no)
+		(fields_autoplaced yes)
+		(property "Reference" "C3"
+			(at 102.87 157.8609 0)
+			(effects
+				(font
+					(size 1.27 1.27)
+				)
+				(justify left)
+			)
+		)
+		(property "Value" "63uF"
+			(at 102.87 160.4009 0)
+			(effects
+				(font
+					(size 1.27 1.27)
+				)
+				(justify left)
+			)
+		)
+		(property "Footprint" ""
+			(at 100.0252 163.83 0)
+			(effects
+				(font
+					(size 1.27 1.27)
+				)
+				(hide yes)
+			)
+		)
+		(property "Datasheet" "~"
+			(at 99.06 160.02 0)
+			(effects
+				(font
+					(size 1.27 1.27)
+				)
+				(hide yes)
+			)
+		)
+		(property "Description" "Polarized capacitor"
+			(at 99.06 160.02 0)
+			(effects
+				(font
+					(size 1.27 1.27)
+				)
+				(hide yes)
+			)
+		)
+		(pin "2"
+		)
+		(pin "1"
+		)
+		(instances
+			(project "Control Board"
+				(path "/0ffd8ca2-c182-4399-851c-8d03eb455740"
+					(reference "C3")
+					(unit 1)
+				)
+			)
+		)
+	)
+	(symbol
 		(lib_id "Regulator_Switching:MC34063AD")
 		(at 72.39 144.78 0)
@@
 			)
 		)
-		(property "Value" "L"
+		(property "Value" "56uH"
 			(at 91.44 147.32 90)
 			(effects
@@
 			)
 		)
-		(property "Value" "R"
+		(property "Value" "11k"
 			(at 114.3 161.2899 0)
 			(effects
@@
 	)
 	(symbol
+		(lib_id "Device:D_Schottky")
+		(at 85.09 160.02 270)
+		(unit 1)
+		(exclude_from_sim no)
+		(in_bom yes)
+		(on_board yes)
+		(dnp no)
+		(fields_autoplaced yes)
+		(property "Reference" "D5"
+			(at 87.63 158.4324 90)
+			(effects
+				(font
+					(size 1.27 1.27)
+				)
+				(justify left)
+			)
+		)
+		(property "Value" "1N5818"
+			(at 87.63 160.9724 90)
+			(effects
+				(font
+					(size 1.27 1.27)
+				)
+				(justify left)
+			)
+		)
+		(property "Footprint" ""
+			(at 85.09 160.02 0)
+			(effects
+				(font
+					(size 1.27 1.27)
+				)
+				(hide yes)
+			)
+		)
+		(property "Datasheet" "~"
+			(at 85.09 160.02 0)
+			(effects
+				(font
+					(size 1.27 1.27)
+				)
+				(hide yes)
+			)
+		)
+		(property "Description" "Schottky diode"
+			(at 85.09 160.02 0)
+			(effects
+				(font
+					(size 1.27 1.27)
+				)
+				(hide yes)
+			)
+		)
+		(pin "1"
+		)
+		(pin "2"
+		)
+		(instances
+			(project "Control Board"
+				(path "/0ffd8ca2-c182-4399-851c-8d03eb455740"
+					(reference "D5")
+					(unit 1)
+				)
+			)
+		)
+	)
+	(symbol
 		(lib_id "Device:R")
 		(at 200.66 46.99 0)
@@
 				(path "/0ffd8ca2-c182-4399-851c-8d03eb455740"
 					(reference "Q5")
-					(unit 1)
-				)
-			)
-		)
-	)
-	(symbol
-		(lib_id "Device:D_Zener")
-		(at 85.09 160.02 270)
-		(unit 1)
-		(exclude_from_sim no)
-		(in_bom yes)
-		(on_board yes)
-		(dnp no)
-		(fields_autoplaced yes)
-		(property "Reference" "D5"
-			(at 87.63 158.7499 90)
-			(effects
-				(font
-					(size 1.27 1.27)
-				)
-				(justify left)
-			)
-		)
-		(property "Value" "D_Zener"
-			(at 87.63 161.2899 90)
-			(effects
-				(font
-					(size 1.27 1.27)
-				)
-				(justify left)
-			)
-		)
-		(property "Footprint" ""
-			(at 85.09 160.02 0)
-			(effects
-				(font
-					(size 1.27 1.27)
-				)
-				(hide yes)
-			)
-		)
-		(property "Datasheet" "~"
-			(at 85.09 160.02 0)
-			(effects
-				(font
-					(size 1.27 1.27)
-				)
-				(hide yes)
-			)
-		)
-		(property "Description" "Zener diode"
-			(at 85.09 160.02 0)
-			(effects
-				(font
-					(size 1.27 1.27)
-				)
-				(hide yes)
-			)
-		)
-		(pin "2"
-		)
-		(pin "1"
-		)
-		(instances
-			(project "Control Board"
-				(path "/0ffd8ca2-c182-4399-851c-8d03eb455740"
-					(reference "D5")
 					(unit 1)
 				)
@@
 					(unit 1)
 				)
-			)
-		)
-	)
-	(symbol
-		(lib_id "Device:C")
-		(at 99.06 160.02 0)
-		(unit 1)
-		(exclude_from_sim no)
-		(in_bom yes)
-		(on_board yes)
-		(dnp no)
-		(fields_autoplaced yes)
-		(property "Reference" "C3"
-			(at 102.87 158.7499 0)
-			(effects
-				(font
-					(size 1.27 1.27)
-				)
-				(justify left)
-			)
-		)
-		(property "Value" "470pF"
-			(at 102.87 161.2899 0)
-			(effects
-				(font
-					(size 1.27 1.27)
-				)
-				(justify left)
-			)
-		)
-		(property "Footprint" ""
-			(at 100.0252 163.83 0)
-			(effects
-				(font
-					(size 1.27 1.27)
-				)
-				(hide yes)
-			)
-		)
-		(property "Datasheet" "~"
-			(at 99.06 160.02 0)
-			(effects
-				(font
-					(size 1.27 1.27)
-				)
-				(hide yes)
-			)
-		)
-		(property "Description" "Unpolarized capacitor"
-			(at 99.06 160.02 0)
-			(effects
-				(font
-					(size 1.27 1.27)
-				)
-				(hide yes)
-			)
-		)
-		(pin "2"
-		)
-		(pin "1"
-		)
-		(instances
-			(project "Control Board"
-				(path "/0ffd8ca2-c182-4399-851c-8d03eb455740"
-					(reference "C3")
-					(unit 1)
-				)
